Commit message: test

File: workspaceRos2/src/phantomx/phantomx_description/urdf/phantomx_urdf.xacro (robot description, xacro)
@@ -42,4 +42,71 @@
         <xacro:leg_l xyz="0 0.1034  0.001116" rpy="0 4.7123 3.14159" suffix="lm"/>
         <xacro:leg_l xyz="-0.1248 0.06164  0.001116" rpy="0 4.7123 3.9269908169872414" suffix="lr"/>
+<joint name="phantomx_camera" type="fixed">
+    <parent link="MP_BODY"/>
+    <child link="camera"/>
+</joint>
+<link name="camera">
+  <inertial>
+    <origin xyz="0 0 0.1"/>
+    <mass value="0.1"/>
+    <inertia ixx="0.2" ixy="0" ixz="0" iyy="0.2" iyz="0"
+             izz="0.2"/>
+  </inertial>
+  <collision name="collision">
+    <geometry>
+      <box>
+        <size>0.073000 0.276000 0.072000</size>
+      </box>
+    </geometry>
+  </collision>
+  <visual name="visual">
+    <geometry>
+      <mesh>
+        <mesh filename="package://phantomx_description/meshes/kinect/meshes/kinect.dae" />
+      </mesh>
+    </geometry>
+  </visual>
+  <sensor name="camera" type="depth">
+    <update_rate>20</update_rate>
+    <camera>
+      <horizontal_fov>1.047198</horizontal_fov>
+      <image>
+        <width>640</width>
+        <height>480</height>
+        <format>R8G8B8</format>
+      </image>
+      <clip>
+        <near>0.05</near>
+        <far>3</far>
+      </clip>
+    </camera>
+    <plugin name="camera_plugin" filename="libgazebo_ros_openni_kinect.so">
+          <baseline>0.2</baseline>
+          <alwaysOn>true</alwaysOn>
+          <!-- Keep this zero, update_rate in the parent <sensor> tag
+            will control the frame rate. -->
+          <updateRate>0.0</updateRate>
+          <cameraName>camera_ir</cameraName>
+          <imageTopicName>/camera/color/image_raw</imageTopicName>
+          <cameraInfoTopicName>/camera/color/camera_info</cameraInfoTopicName>
+          <depthImageTopicName>/camera/depth/image_raw</depthImageTopicName>
+          <depthImageCameraInfoTopicName>/camera/depth/camera_info</depthImageCameraInfoTopicName>
+          <pointCloudTopicName>/camera/depth/points</pointCloudTopicName>
+          <frameName>camera_link</frameName>
+          <pointCloudCutoff>0.5</pointCloudCutoff>
+          <pointCloudCutoffMax>3.0</pointCloudCutoffMax>
+          <distortionK1>0</distortionK1>
+          <distortionK2>0</distortionK2>
+          <distortionK3>0</distortionK3>
+          <distortionT1>0</distortionT1>
+          <distortionT2>0</distortionT2>
+          <CxPrime>0</CxPrime>
+          <Cx>0</Cx>
+          <Cy>0</Cy>
+          <focalLength>0</focalLength>
+          <hackBaseline>0</hackBaseline>
+        </plugin>
+  </sensor>
+</link>
     </xacro:macro>
     <xacro:macro name="leg_l" params="xyz rpy suffix">

Commit message: OK

File: workspaceRos2/src/phantomx/phantomx_description/urdf/phantomx_urdf.xacro (robot description, xacro)
@@ -42,30 +42,36 @@
         <xacro:leg_l xyz="0 0.1034  0.001116" rpy="0 4.7123 3.14159" suffix="lm"/>
         <xacro:leg_l xyz="-0.1248 0.06164  0.001116" rpy="0 4.7123 3.9269908169872414" suffix="lr"/>
-<joint name="phantomx_camera" type="fixed">
+      <xacro:camera2 xyz="0 -0.08164  0.102" rpy="0 0 -1.5707" suffix="right"/>
+      <xacro:camera2 xyz="0 0.08164  0.102" rpy="0 0 1.5707" suffix="left"/>
+    </xacro:macro>
+ <xacro:macro name="camera2" params="xyz rpy suffix">
+<joint name="phantomx_camera_${suffix}" type="fixed">
     <parent link="MP_BODY"/>
-    <child link="camera"/>
+    <child link="camera_${suffix}"/>
+    <origin xyz="${xyz}" rpy="${rpy}" />
 </joint>
-<link name="camera">
+<link name="camera_${suffix}">
   <inertial>
-    <origin xyz="0 0 0.1"/>
+    <origin xyz="0 0 0" rpy="0 0 0"/>
     <mass value="0.1"/>
     <inertia ixx="0.2" ixy="0" ixz="0" iyy="0.2" iyz="0"
              izz="0.2"/>
   </inertial>
-  <collision name="collision">
+  <collision>
+    <origin xyz="0 0 0" rpy="0 0 0"/>
     <geometry>
-      <box>
-        <size>0.073000 0.276000 0.072000</size>
-      </box>
+      <box size="0.073000 0.276000 0.072000"/>
     </geometry>
   </collision>
-  <visual name="visual">
+  <visual>
+    <origin xyz="0 0 0" rpy="0 0 0"/>
     <geometry>
-      <mesh>
-        <mesh filename="package://phantomx_description/meshes/kinect/meshes/kinect.dae" />
-      </mesh>
+         <!--<box size="0.073000 0.276000 0.072000"/>-->
+         <mesh filename="package://phantomx_description/meshes/kinect/meshes/kinect.dae" />-->
     </geometry>
   </visual>
-  <sensor name="camera" type="depth">
+</link>
+<gazebo reference="camera_${suffix}">
+ <sensor name="camera_{suffix}" type="depth">
     <update_rate>20</update_rate>
     <camera>
@@ -84,14 +90,12 @@
           <baseline>0.2</baseline>
           <alwaysOn>true</alwaysOn>
-          <!-- Keep this zero, update_rate in the parent <sensor> tag
-            will control the frame rate. -->
           <updateRate>0.0</updateRate>
-          <cameraName>camera_ir</cameraName>
-          <imageTopicName>/camera/color/image_raw</imageTopicName>
-          <cameraInfoTopicName>/camera/color/camera_info</cameraInfoTopicName>
-          <depthImageTopicName>/camera/depth/image_raw</depthImageTopicName>
-          <depthImageCameraInfoTopicName>/camera/depth/camera_info</depthImageCameraInfoTopicName>
-          <pointCloudTopicName>/camera/depth/points</pointCloudTopicName>
-          <frameName>camera_link</frameName>
+          <cameraName>camera_${suffix}</cameraName>
+          <imageTopicName>/phantomx/camera_${suffix}/color/image_raw</imageTopicName>
+          <cameraInfoTopicName>/phantomx/camera_${suffix}/color/camera_info</cameraInfoTopicName>
+          <depthImageTopicName>/phantomx/camera_${suffix}/depth/image_raw</depthImageTopicName>
+          <depthImageCameraInfoTopicName>/phantomx/camera_${suffix}/depth/camera_info</depthImageCameraInfoTopicName>
+          <pointCloudTopicName>/phantomx/camera_${suffix}/depth/points</pointCloudTopicName>
+          <frameName>camera_${suffix}</frameName>
           <pointCloudCutoff>0.5</pointCloudCutoff>
           <pointCloudCutoffMax>3.0</pointCloudCutoffMax>
@@ -108,6 +112,6 @@
         </plugin>
   </sensor>
-</link>
-    </xacro:macro>
+</gazebo>
+</xacro:macro>
     <xacro:macro name="leg_l" params="xyz rpy suffix">
         <link name="c1_${suffix}">

Commit message: ok devel

File: workspaceRos2/src/phantomx/phantomx_description/urdf/phantomx_urdf.xacro (robot description, xacro)
@@ -42,30 +42,36 @@
         <xacro:leg_l xyz="0 0.1034  0.001116" rpy="0 4.7123 3.14159" suffix="lm"/>
         <xacro:leg_l xyz="-0.1248 0.06164  0.001116" rpy="0 4.7123 3.9269908169872414" suffix="lr"/>
-<joint name="phantomx_camera" type="fixed">
+      <xacro:camera2 xyz="0 -0.08164  0.142" rpy="0 0 -1.5707" suffix="right"/>
+      <xacro:camera2 xyz="0 0.08164  0.142" rpy="0 0 1.5707" suffix="left"/>
+    </xacro:macro>
+ <xacro:macro name="camera2" params="xyz rpy suffix">
+<joint name="phantomx_camera_${suffix}" type="fixed">
     <parent link="MP_BODY"/>
-    <child link="camera"/>
+    <child link="camera_${suffix}"/>
+    <origin xyz="${xyz}" rpy="${rpy}" />
 </joint>
-<link name="camera">
+<link name="camera_${suffix}">
   <inertial>
-    <origin xyz="0 0 0.1"/>
+    <origin xyz="0 0 0" rpy="0 0 0"/>
     <mass value="0.1"/>
     <inertia ixx="0.2" ixy="0" ixz="0" iyy="0.2" iyz="0"
              izz="0.2"/>
   </inertial>
-  <collision name="collision">
+  <collision>
+    <origin xyz="0 0 0" rpy="0 0 0"/>
     <geometry>
-      <box>
-        <size>0.073000 0.276000 0.072000</size>
-      </box>
+      <box size="0.073000 0.276000 0.072000"/>
     </geometry>
   </collision>
-  <visual name="visual">
+  <visual>
+    <origin xyz="0 0 0" rpy="0 0 0"/>
     <geometry>
-      <mesh>
-        <mesh filename="package://phantomx_description/meshes/kinect/meshes/kinect.dae" />
-      </mesh>
+         <!--<box size="0.073000 0.276000 0.072000"/>-->
+         <mesh filename="package://phantomx_description/meshes/kinect/meshes/kinect.dae" />-->
     </geometry>
   </visual>
-  <sensor name="camera" type="depth">
+</link>
+<gazebo reference="camera_${suffix}">
+ <sensor name="camera_{suffix}" type="depth">
     <update_rate>20</update_rate>
     <camera>
@@ -84,14 +90,12 @@
           <baseline>0.2</baseline>
           <alwaysOn>true</alwaysOn>
-          <!-- Keep this zero, update_rate in the parent <sensor> tag
-            will control the frame rate. -->
           <updateRate>0.0</updateRate>
-          <cameraName>camera_ir</cameraName>
-          <imageTopicName>/camera/color/image_raw</imageTopicName>
-          <cameraInfoTopicName>/camera/color/camera_info</cameraInfoTopicName>
-          <depthImageTopicName>/camera/depth/image_raw</depthImageTopicName>
-          <depthImageCameraInfoTopicName>/camera/depth/camera_info</depthImageCameraInfoTopicName>
-          <pointCloudTopicName>/camera/depth/points</pointCloudTopicName>
-          <frameName>camera_link</frameName>
+          <cameraName>camera_${suffix}</cameraName>
+          <imageTopicName>/phantomx/camera_${suffix}/color/image_raw</imageTopicName>
+          <cameraInfoTopicName>/phantomx/camera_${suffix}/color/camera_info</cameraInfoTopicName>
+          <depthImageTopicName>/phantomx/camera_${suffix}/depth/image_raw</depthImageTopicName>
+          <depthImageCameraInfoTopicName>/phantomx/camera_${suffix}/depth/camera_info</depthImageCameraInfoTopicName>
+          <pointCloudTopicName>/phantomx/camera_${suffix}/depth/points</pointCloudTopicName>
+          <frameName>camera_${suffix}</frameName>
           <pointCloudCutoff>0.5</pointCloudCutoff>
           <pointCloudCutoffMax>3.0</pointCloudCutoffMax>
@@ -108,6 +112,6 @@
         </plugin>
   </sensor>
-</link>
-    </xacro:macro>
+</gazebo>
+</xacro:macro>
     <xacro:macro name="leg_l" params="xyz rpy suffix">
         <link name="c1_${suffix}">

Commit message: Add new camera

File: workspaceRos2/src/phantomx/phantomx_description/urdf/phantomx_urdf.xacro (robot description, xacro)
@@ -42,74 +42,77 @@
         <xacro:leg_l xyz="0 0.1034  0.001116" rpy="0 4.7123 3.14159" suffix="lm"/>
         <xacro:leg_l xyz="-0.1248 0.06164  0.001116" rpy="0 4.7123 3.9269908169872414" suffix="lr"/>
-      <xacro:camera2 xyz="0 -0.08164  0.142" rpy="0 0 -1.5707" suffix="right"/>
-      <xacro:camera2 xyz="0 0.08164  0.142" rpy="0 0 1.5707" suffix="left"/>
+<!-- <xacro:camera2 xyz="0 -0.08164  0.142" rpy="0 0 -1.5707" suffix="right"/>
+ <xacro:camera2 xyz="0 0.08164  0.142" rpy="0 0 1.5707" suffix="left"/> -->
+ <xacro:camera2 xyz="-0.1 -0.08164  0.142" rpy="0 -0.52 -1.5707" suffix="right"/>
+ <xacro:camera2 xyz="-0.1 0.08164  0.142" rpy="0 -0.52 1.5707" suffix="left"/>
+ <xacro:camera2 xyz="0.125 0  0.142" rpy="0 -0.52 0" suffix="front"/>
 </xacro:macro>
 <xacro:macro name="camera2" params="xyz rpy suffix">
 <joint name="phantomx_camera_${suffix}" type="fixed">
-    <parent link="MP_BODY"/>
-    <child link="camera_${suffix}"/>
-    <origin xyz="${xyz}" rpy="${rpy}" />
+<parent link="MP_BODY"/>
+<child link="camera_${suffix}"/>
+<origin xyz="${xyz}" rpy="${rpy}" />
 </joint>
 <link name="camera_${suffix}">
-  <inertial>
-    <origin xyz="0 0 0" rpy="0 0 0"/>
-    <mass value="0.1"/>
-    <inertia ixx="0.2" ixy="0" ixz="0" iyy="0.2" iyz="0"
-             izz="0.2"/>
-  </inertial>
-  <collision>
-    <origin xyz="0 0 0" rpy="0 0 0"/>
-    <geometry>
-      <box size="0.073000 0.276000 0.072000"/>
-    </geometry>
-  </collision>
-  <visual>
-    <origin xyz="0 0 0" rpy="0 0 0"/>
-    <geometry>
-         <!--<box size="0.073000 0.276000 0.072000"/>-->
-         <mesh filename="package://phantomx_description/meshes/kinect/meshes/kinect.dae" />-->
-    </geometry>
-  </visual>
+<inertial>
+<origin xyz="0 0 0" rpy="0 0 0"/>
+<mass value="0.1"/>
+<inertia ixx="0.2" ixy="0" ixz="0" iyy="0.2" iyz="0"
+        izz="0.2"/>
+</inertial>
+<collision>
+<origin xyz="0 0 0" rpy="0 0 0"/>
+<geometry>
+ <box size="0.073000 0.276000 0.072000"/>
+</geometry>
+</collision>
+<visual>
+<origin xyz="0 0 0" rpy="0 0 0"/>
+<geometry>
+    <!--<box size="0.073000 0.276000 0.072000"/>-->
+    <mesh filename="package://phantomx_description/meshes/kinect/meshes/kinect.dae" />-->
+</geometry>
+</visual>
 </link>
 <gazebo reference="camera_${suffix}">
- <sensor name="camera_{suffix}" type="depth">
-    <update_rate>20</update_rate>
-    <camera>
-      <horizontal_fov>1.047198</horizontal_fov>
-      <image>
-        <width>640</width>
-        <height>480</height>
-        <format>R8G8B8</format>
-      </image>
-      <clip>
-        <near>0.05</near>
-        <far>3</far>
-      </clip>
-    </camera>
-    <plugin name="camera_plugin" filename="libgazebo_ros_openni_kinect.so">
-          <baseline>0.2</baseline>
-          <alwaysOn>true</alwaysOn>
-          <updateRate>0.0</updateRate>
-          <cameraName>camera_${suffix}</cameraName>
-          <imageTopicName>/phantomx/camera_${suffix}/color/image_raw</imageTopicName>
-          <cameraInfoTopicName>/phantomx/camera_${suffix}/color/camera_info</cameraInfoTopicName>
-          <depthImageTopicName>/phantomx/camera_${suffix}/depth/image_raw</depthImageTopicName>
-          <depthImageCameraInfoTopicName>/phantomx/camera_${suffix}/depth/camera_info</depthImageCameraInfoTopicName>
-          <pointCloudTopicName>/phantomx/camera_${suffix}/depth/points</pointCloudTopicName>
-          <frameName>camera_${suffix}</frameName>
-          <pointCloudCutoff>0.5</pointCloudCutoff>
-          <pointCloudCutoffMax>3.0</pointCloudCutoffMax>
-          <distortionK1>0</distortionK1>
-          <distortionK2>0</distortionK2>
-          <distortionK3>0</distortionK3>
-          <distortionT1>0</distortionT1>
-          <distortionT2>0</distortionT2>
-          <CxPrime>0</CxPrime>
-          <Cx>0</Cx>
-          <Cy>0</Cy>
-          <focalLength>0</focalLength>
-          <hackBaseline>0</hackBaseline>
-        </plugin>
-  </sensor>
+<sensor name="camera_{suffix}" type="depth">
+<update_rate>20</update_rate>
+<camera>
+ <horizontal_fov>1.047198</horizontal_fov>
+ <image>
+   <width>640</width>
+   <height>480</height>
+   <format>R8G8B8</format>
+ </image>
+ <clip>
+   <near>0.05</near>
+   <far>10</far>
+ </clip>
+</camera>
+<plugin name="camera_plugin" filename="libgazebo_ros_openni_kinect.so">
+     <baseline>0.2</baseline>
+     <alwaysOn>true</alwaysOn>
+     <updateRate>0.0</updateRate>
+     <cameraName>camera_${suffix}</cameraName>
+     <imageTopicName>/phantomx/camera_${suffix}/color/image_raw</imageTopicName>
+     <cameraInfoTopicName>/phantomx/camera_${suffix}/color/camera_info</cameraInfoTopicName>
+     <depthImageTopicName>/phantomx/camera_${suffix}/depth/image_raw</depthImageTopicName>
+     <depthImageCameraInfoTopicName>/phantomx/camera_${suffix}/depth/camera_info</depthImageCameraInfoTopicName>
+     <pointCloudTopicName>/phantomx/camera_${suffix}/depth/points</pointCloudTopicName>
+     <frameName>camera_${suffix}</frameName>
+     <pointCloudCutoff>0.1</pointCloudCutoff>
+     <pointCloudCutoffMax>2.0</pointCloudCutoffMax>
+     <distortionK1>0</distortionK1>
+     <distortionK2>0</distortionK2>
+     <distortionK3>0</distortionK3>
+     <distortionT1>0</distortionT1>
+     <distortionT2>0</distortionT2>
+     <CxPrime>0</CxPrime>
+     <Cx>0</Cx>
+     <Cy>0</Cy>
+     <focalLength>0</focalLength>
+     <hackBaseline>0</hackBaseline>
+   </plugin>
+</sensor>
 </gazebo>
 </xacro:macro>
@@ -315,5 +318,5 @@
         </geometry>
         <material name="Cyan">
-  14        <color rgba="0 1.0 1.0 1.0"/>
+          <color rgba="0 1.0 1.0 1.0"/>
         </material>
       </visual>
